Commit message: Fix URDF orientations for Gazebo, add joint motion simulator, and update ROS 2 launch scripts

File: urdf/unnamed/urdf/unnamed_gazebo.urdf (robot description, URDF)
Before this commit: robot unnamed, 13 links, 12 joints
Links:
- removed link Gripper+Rod+Geared_left_link
- removed link Gripper+Rod+Geared_right_link
- removed link Gripper+finger+Geared_left_link
- removed link Gripper+finger+Geared_right_link
- removed link gripper_base_link
- removed link left_parallel_link
- removed link right_parallel_link
Joints:
- removed joint Gripper+finger+Geared_left_joint
- removed joint Gripper+finger+Geared_right_joint
- removed joint left_parallel_link_joint
- removed joint right_parallel_link_joint
- removed joint turntable_link_joint_dup_3
- removed joint turntable_link_joint_dup_4
- removed joint turntable_link_joint_dup_5
- joint turntable_link_joint: origin xyz=-0.031938 -0.000753 0.048262 rpy=0 0 0 -> xyz=-0.029849 -0.000704 0.045105 rpy=0 0 3.13716
- joint turntable_link_joint_dup: origin xyz=-0.048477 -0.000318 0.048276 rpy=0 0 0 -> xyz=-0.045306 -0.000297 0.045118 rpy=0 0 0.00443
- joint turntable_link_joint_dup_1: origin xyz=0.050543 -0.001967 0.208029 rpy=0 0 0 -> xyz=0.047192 -0.001837 0.194238 rpy=1.57078 1.56581 1.57078
- joint turntable_link_joint_dup_2: origin xyz=-0.000158 -0.000855 0.152797 rpy=0 0 0 -> xyz=-0.000145 -0.000782 0.139796 rpy=0.00167 0.01634 0.01070
