Commit message: Add web dashboard, joint calibration GUI, servo commander, and update hardware integration

File: urdf/unnamed/urdf/unnamed.urdf (robot description, URDF)
Before this commit: robot unnamed, 12 links, 11 joints
Joints:
- joint Gripper+finger+Geared_left_link: axis (none) -> 0.00000 0.00000 1.00000; limit (none) -> lower=-2.00000 upper=2.00000 effort=0.00000 velocity=0.00000
- joint Gripper+finger+Geared_right_link: axis (none) -> 0.00000 0.00000 1.00000; limit (none) -> lower=-2.00000 upper=2.00000 effort=0.00000 velocity=0.00000

Commit message: feat: Implement upper-body gesture teleoperation and unified dashboard mode switching
- Add gesture_teleop_node with MediaPipe upper-body tracking (strictly till waist level) and cyberpunk HUD overlay.
- Integrate 1-click 'Gesture Mode' toggle button into PyQt5 Control Panel (calibrated_joint_gui.py).
- Fix RViz dual-publishing topic collision and restore photorealistic 3D CAD STL mesh rendering.
- Add low-sensitivity EMA filtering (alpha=0.10), 1.5° deadbanding, and defined posture zone detection.
- Add standalone gesture launcher script launch_gesture_teleop.sh.

File: urdf/unnamed/urdf/unnamed.urdf (robot description, URDF)
Before this commit: robot unnamed, 12 links, 11 joints
Links:
- link Elbow_1_link: geometry visual mesh filename=file:///home/chakradhar/Documents/Hardware/urdf/unnamed/mes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 scale=0.00100 0.00100 0.00100
- link Elbow_2_link: geometry visual mesh filename=file:///home/chakradhar/Documents/Hardware/urdf/unnamed/mes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 scale=0.00100 0.00100 0.00100
- link Gripper+Rod+Geared_left_link: geometry visual mesh filename=file:///home/chakradhar/Documents/Hardware/urdf/unnamed/mes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 scale=-0.00100 -0.00100 -0.00100
- link Gripper+Rod+Geared_right_link: geometry visual mesh filename=file:///home/chakradhar/Documents/Hardware/urdf/unnamed/mes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 scale=0.00100 -0.00100 -0.00100
- link Gripper+finger+Geared_left_link: geometry visual mesh filename=file:///home/chakradhar/Documents/Hardware/urdf/unnamed/mes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 scale=-0.00100 -0.00100 -0.00100
- link Gripper+finger+Geared_right_link: geometry visual mesh filename=file:///home/chakradhar/Documents/Hardware/urdf/unnamed/mes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 scale=0.00100 -0.00100 -0.00100
- link Wrist_pitch._link: geometry visual mesh filename=file:///home/chakradhar/Documents/Hardware/urdf/unnamed/mes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 scale=0.00100 0.00100 0.00100
- link basecase1_link: geometry visual mesh filename=file:///home/chakradhar/Documents/Hardware/urdf/unnamed/mes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 scale=0.00100 0.00100 0.00100
- link gripper_base_link: geometry visual mesh filename=file:///home/chakradhar/Documents/Hardware/urdf/unnamed/mes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 scale=0.00100 0.00100 -0.00100
- link left_parallel_link: geometry visual mesh filename=file:///home/chakradhar/Documents/Hardware/urdf/unnamed/mes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 scale=-0.00100 -0.00100 -0.00100
- link right_parallel_link: geometry visual mesh filename=file:///home/chakradhar/Documents/Hardware/urdf/unnamed/mes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 scale=0.00100 -0.00100 -0.00100
- link turntable_link: geometry visual mesh filename=file:///home/chakradhar/Documents/Hardware/urdf/unnamed/mes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 scale=0.00100 0.00100 0.00100

File: urdf/unnamed/urdf/unnamed_gazebo.urdf (robot description, URDF)
Before this commit: robot unnamed, 6 links, 5 joints
Links:
- link Elbow_1_link: geometry collision mesh filename=file:///home/chakradhar/Documents/Hardware/urdf/unnamed/mes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 scale=0.00100 0.00100 0.00100; visual mesh filename=file:///home/chakradhar/Documents/Hardware/urdf/unnamed/mes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 scale=0.00100 0.00100 0.00100
- link Elbow_2_link: geometry collision mesh filename=file:///home/chakradhar/Documents/Hardware/urdf/unnamed/mes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 scale=0.00100 0.00100 0.00100; visual mesh filename=file:///home/chakradhar/Documents/Hardware/urdf/unnamed/mes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 scale=0.00100 0.00100 0.00100
- link Wrist_pitch._link: geometry collision mesh filename=file:///home/chakradhar/Documents/Hardware/urdf/unnamed/mes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 scale=0.00100 0.00100 0.00100; visual mesh filename=file:///home/chakradhar/Documents/Hardware/urdf/unnamed/mes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 scale=0.00100 0.00100 0.00100
- link basecase1_link: geometry collision mesh filename=file:///home/chakradhar/Documents/Hardware/urdf/unnamed/mes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 scale=0.00100 0.00100 0.00100; visual mesh filename=file:///home/chakradhar/Documents/Hardware/urdf/unnamed/mes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 scale=0.00100 0.00100 0.00100
- link turntable_link: geometry collision mesh filename=file:///home/chakradhar/Documents/Hardware/urdf/unnamed/mes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 scale=0.00100 0.00100 0.00100; visual mesh filename=file:///home/chakradhar/Documents/Hardware/urdf/unnamed/mes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 scale=0.00100 0.00100 0.00100

File: urdf/unnamed/urdf/unnamed_scaled.urdf (robot description, URDF)
Before this commit: robot unnamed, 13 links, 12 joints
Links:
- link Elbow_1_link: geometry collision mesh filename=file:///home/chakradhar/Documents/Hardware/urdf/unnamed/mes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 scale=0.00100 0.00100 0.00100; visual mesh filename=file:///home/chakradhar/Documents/Hardware/urdf/unnamed/mes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 scale=0.00100 0.00100 0.00100
- link Elbow_2_link: geometry collision mesh filename=file:///home/chakradhar/Documents/Hardware/urdf/unnamed/mes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 scale=0.00100 0.00100 0.00100; visual mesh filename=file:///home/chakradhar/Documents/Hardware/urdf/unnamed/mes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 scale=0.00100 0.00100 0.00100
- link Gripper+Rod+Geared_left_link: geometry collision mesh filename=file:///home/chakradhar/Documents/Hardware/urdf/unnamed/mes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 scale=-0.00100 -0.00100 -0.00100; visual mesh filename=file:///home/chakradhar/Documents/Hardware/urdf/unnamed/mes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 scale=-0.00100 -0.00100 -0.00100
- link Gripper+Rod+Geared_right_link: geometry collision mesh filename=file:///home/chakradhar/Documents/Hardware/urdf/unnamed/mes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 scale=0.00100 -0.00100 -0.00100; visual mesh filename=file:///home/chakradhar/Documents/Hardware/urdf/unnamed/mes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 scale=0.00100 -0.00100 -0.00100
- link Gripper+finger+Geared_left_link: geometry collision mesh filename=file:///home/chakradhar/Documents/Hardware/urdf/unnamed/mes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 scale=-0.00100 -0.00100 -0.00100; visual mesh filename=file:///home/chakradhar/Documents/Hardware/urdf/unnamed/mes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 scale=-0.00100 -0.00100 -0.00100
- link Gripper+finger+Geared_right_link: geometry collision mesh filename=file:///home/chakradhar/Documents/Hardware/urdf/unnamed/mes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 scale=0.00100 -0.00100 -0.00100; visual mesh filename=file:///home/chakradhar/Documents/Hardware/urdf/unnamed/mes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 scale=0.00100 -0.00100 -0.00100
- link Wrist_pitch._link: geometry collision mesh filename=file:///home/chakradhar/Documents/Hardware/urdf/unnamed/mes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 scale=0.00100 0.00100 0.00100; visual mesh filename=file:///home/chakradhar/Documents/Hardware/urdf/unnamed/mes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 scale=0.00100 0.00100 0.00100
- link basecase1_link: geometry collision mesh filename=file:///home/chakradhar/Documents/Hardware/urdf/unnamed/mes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 scale=0.00100 0.00100 0.00100; visual mesh filename=file:///home/chakradhar/Documents/Hardware/urdf/unnamed/mes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 scale=0.00100 0.00100 0.00100
- link gripper_base_link: geometry collision mesh filename=file:///home/chakradhar/Documents/Hardware/urdf/unnamed/mes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 scale=0.00100 0.00100 -0.00100; visual mesh filename=file:///home/chakradhar/Documents/Hardware/urdf/unnamed/mes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 scale=0.00100 0.00100 -0.00100
- link left_parallel_link: geometry collision mesh filename=file:///home/chakradhar/Documents/Hardware/urdf/unnamed/mes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 scale=-0.00100 -0.00100 -0.00100; visual mesh filename=file:///home/chakradhar/Documents/Hardware/urdf/unnamed/mes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 scale=-0.00100 -0.00100 -0.00100
- link right_parallel_link: geometry collision mesh filename=file:///home/chakradhar/Documents/Hardware/urdf/unnamed/mes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 scale=0.00100 -0.00100 -0.00100; visual mesh filename=file:///home/chakradhar/Documents/Hardware/urdf/unnamed/mes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 scale=0.00100 -0.00100 -0.00100
- link turntable_link: geometry collision mesh filename=file:///home/chakradhar/Documents/Hardware/urdf/unnamed/mes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 scale=0.00100 0.00100 0.00100; visual mesh filename=file:///home/chakradhar/Documents/Hardware/urdf/unnamed/mes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 scale=0.00100 0.00100 0.00100

Commit message: Update hardcoded paths to new workspace location and add new servo ESP8266 file

File: urdf/unnamed/urdf/unnamed.urdf (robot description, URDF)
Before this commit: robot unnamed, 12 links, 11 joints
Links:
- link Elbow_1_link: geometry visual mesh filename=file:///home/sabo/Documents/learn_/Hardware/urdf/unnamed/me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 scale=0.00100 0.00100 0.00100
- link Elbow_2_link: geometry visual mesh filename=file:///home/sabo/Documents/learn_/Hardware/urdf/unnamed/me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 scale=0.00100 0.00100 0.00100
- link Gripper+Rod+Geared_left_link: geometry visual mesh filename=file:///home/sabo/Documents/learn_/Hardware/urdf/unnamed/me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 scale=-0.00100 -0.00100 -0.00100
- link Gripper+Rod+Geared_right_link: geometry visual mesh filename=file:///home/sabo/Documents/learn_/Hardware/urdf/unnamed/me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 scale=0.00100 -0.00100 -0.00100
- link Gripper+finger+Geared_left_link: geometry visual mesh filename=file:///home/sabo/Documents/learn_/Hardware/urdf/unnamed/me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 scale=-0.00100 -0.00100 -0.00100
- link Gripper+finger+Geared_right_link: geometry visual mesh filename=file:///home/sabo/Documents/learn_/Hardware/urdf/unnamed/me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 scale=0.00100 -0.00100 -0.00100
- link Wrist_pitch._link: geometry visual mesh filename=file:///home/sabo/Documents/learn_/Hardware/urdf/unnamed/me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 scale=0.00100 0.00100 0.00100
- link basecase1_link: geometry visual mesh filename=file:///home/sabo/Documents/learn_/Hardware/urdf/unnamed/me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 scale=0.00100 0.00100 0.00100
- link gripper_base_link: geometry visual mesh filename=file:///home/sabo/Documents/learn_/Hardware/urdf/unnamed/me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 scale=0.00100 0.00100 -0.00100
- link left_parallel_link: geometry visual mesh filename=file:///home/sabo/Documents/learn_/Hardware/urdf/unnamed/me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 scale=-0.00100 -0.00100 -0.00100
- link right_parallel_link: geometry visual mesh filename=file:///home/sabo/Documents/learn_/Hardware/urdf/unnamed/me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 scale=0.00100 -0.00100 -0.00100
- link turntable_link: geometry visual mesh filename=file:///home/sabo/Documents/learn_/Hardware/urdf/unnamed/me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 scale=0.00100 0.00100 0.00100

File: urdf/unnamed/urdf/unnamed_gazebo.urdf (robot description, URDF)
Before this commit: robot unnamed, 6 links, 5 joints
Links:
- link Elbow_1_link: geometry collision mesh filename=file:///home/sabo/Documents/learn_/Hardware/urdf/unnamed/me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 scale=0.00100 0.00100 0.00100; visual mesh filename=file:///home/sabo/Documents/learn_/Hardware/urdf/unnamed/me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 scale=0.00100 0.00100 0.00100
- link Elbow_2_link: geometry collision mesh filename=file:///home/sabo/Documents/learn_/Hardware/urdf/unnamed/me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 scale=0.00100 0.00100 0.00100; visual mesh filename=file:///home/sabo/Documents/learn_/Hardware/urdf/unnamed/me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 scale=0.00100 0.00100 0.00100
- link Wrist_pitch._link: geometry collision mesh filename=file:///home/sabo/Documents/learn_/Hardware/urdf/unnamed/me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 scale=0.00100 0.00100 0.00100; visual mesh filename=file:///home/sabo/Documents/learn_/Hardware/urdf/unnamed/me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 scale=0.00100 0.00100 0.00100
- link basecase1_link: geometry collision mesh filename=file:///home/sabo/Documents/learn_/Hardware/urdf/unnamed/me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 scale=0.00100 0.00100 0.00100; visual mesh filename=file:///home/sabo/Documents/learn_/Hardware/urdf/unnamed/me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 scale=0.00100 0.00100 0.00100
- link turntable_link: geometry collision mesh filename=file:///home/sabo/Documents/learn_/Hardware/urdf/unnamed/me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 scale=0.00100 0.00100 0.00100; visual mesh filename=file:///home/sabo/Documents/learn_/Hardware/urdf/unnamed/me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 scale=0.00100 0.00100 0.00100

File: urdf/unnamed/urdf/unnamed_scaled.urdf (robot description, URDF)
Before this commit: robot unnamed, 13 links, 12 joints
Links:
- link Elbow_1_link: geometry collision mesh filename=file:///home/sabo/Documents/learn_/Hardware/urdf/unnamed/me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 scale=0.00100 0.00100 0.00100; visual mesh filename=file:///home/sabo/Documents/learn_/Hardware/urdf/unnamed/me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 scale=0.00100 0.00100 0.00100
- link Elbow_2_link: geometry collision mesh filename=file:///home/sabo/Documents/learn_/Hardware/urdf/unnamed/me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 scale=0.00100 0.00100 0.00100; visual mesh filename=file:///home/sabo/Documents/learn_/Hardware/urdf/unnamed/me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 scale=0.00100 0.00100 0.00100
- link Gripper+Rod+Geared_left_link: geometry collision mesh filename=file:///home/sabo/Documents/learn_/Hardware/urdf/unnamed/me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 scale=-0.00100 -0.00100 -0.00100; visual mesh filename=file:///home/sabo/Documents/learn_/Hardware/urdf/unnamed/me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 scale=-0.00100 -0.00100 -0.00100
- link Gripper+Rod+Geared_right_link: geometry collision mesh filename=file:///home/sabo/Documents/learn_/Hardware/urdf/unnamed/me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 scale=0.00100 -0.00100 -0.00100; visual mesh filename=file:///home/sabo/Documents/learn_/Hardware/urdf/unnamed/me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 scale=0.00100 -0.00100 -0.00100
- link Gripper+finger+Geared_left_link: geometry collision mesh filename=file:///home/sabo/Documents/learn_/Hardware/urdf/unnamed/me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 scale=-0.00100 -0.00100 -0.00100; visual mesh filename=file:///home/sabo/Documents/learn_/Hardware/urdf/unnamed/me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 scale=-0.00100 -0.00100 -0.00100
- link Gripper+finger+Geared_right_link: geometry collision mesh filename=file:///home/sabo/Documents/learn_/Hardware/urdf/unnamed/me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 scale=0.00100 -0.00100 -0.00100; visual mesh filename=file:///home/sabo/Documents/learn_/Hardware/urdf/unnamed/me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 scale=0.00100 -0.00100 -0.00100
- link Wrist_pitch._link: geometry collision mesh filename=file:///home/sabo/Documents/learn_/Hardware/urdf/unnamed/me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 scale=0.00100 0.00100 0.00100; visual mesh filename=file:///home/sabo/Documents/learn_/Hardware/urdf/unnamed/me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 scale=0.00100 0.00100 0.00100
- link basecase1_link: geometry collision mesh filename=file:///home/sabo/Documents/learn_/Hardware/urdf/unnamed/me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 scale=0.00100 0.00100 0.00100; visual mesh filename=file:///home/sabo/Documents/learn_/Hardware/urdf/unnamed/me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 scale=0.00100 0.00100 0.00100
- link gripper_base_link: geometry collision mesh filename=file:///home/sabo/Documents/learn_/Hardware/urdf/unnamed/me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 scale=0.00100 0.00100 -0.00100; visual mesh filename=file:///home/sabo/Documents/learn_/Hardware/urdf/unnamed/me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 scale=0.00100 0.00100 -0.00100
- link left_parallel_link: geometry collision mesh filename=file:///home/sabo/Documents/learn_/Hardware/urdf/unnamed/me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 scale=-0.00100 -0.00100 -0.00100; visual mesh filename=file:///home/sabo/Documents/learn_/Hardware/urdf/unnamed/me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 scale=-0.00100 -0.00100 -0.00100
- link right_parallel_link: geometry collision mesh filename=file:///home/sabo/Documents/learn_/Hardware/urdf/unnamed/me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 scale=0.00100 -0.00100 -0.00100; visual mesh filename=file:///home/sabo/Documents/learn_/Hardware/urdf/unnamed/me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 scale=0.00100 -0.00100 -0.00100
- link turntable_link: geometry collision mesh filename=file:///home/sabo/Documents/learn_/Hardware/urdf/unnamed/me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 scale=0.00100 0.00100 0.00100; visual mesh filename=file:///home/sabo/Documents/learn_/Hardware/urdf/unnamed/me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 scale=0.00100 0.00100 0.00100

Commit message: feat: Add quadruped robot model, URDF/smurf export configs, and enhance dashboard RViz embedding

File: urdf/unnamed/urdf/unnamed.urdf (robot description, URDF)
Before this commit: robot unnamed, 12 links, 11 joints
Links:
- removed link Elbow_1_link
- removed link Elbow_2_link
- removed link Gripper+Rod+Geared_left_link
- removed link Gripper+Rod+Geared_right_link
- removed link Gripper+finger+Geared_left_link
- removed link Gripper+finger+Geared_right_link
- removed link Wrist_pitch._link
- removed link basecase1_link
- removed link gripper_base_link
- removed link left_parallel_link
- removed link right_parallel_link
- removed link turntable_link
- added link Internal-Frame-v121_link
- added link L1-v117_link
- added link L2-v117_link
- added link L3-v117_link
- added link L4-v117_link
- added link R1-v117_link
- added link R2-v117_link
- added link R3-v117_link
- added link R4-v117_link
Joints:
- removed joint Gripper+finger+Geared_left_link
- removed joint Gripper+finger+Geared_right_link
- removed joint left_parallel_link_joint
- removed joint right_parallel_link_joint
- removed joint turntable_link_joint
- removed joint turntable_link_joint_dup
- removed joint turntable_link_joint_dup_1
- removed joint turntable_link_joint_dup_2
- removed joint turntable_link_joint_dup_3
- removed joint turntable_link_joint_dup_4
- removed joint turntable_link_joint_dup_5
- added joint R3-v117_link_joint: type revolute, parent R1-v117_link, child R3-v117_link, origin xyz=-0.94144 -3.68561 -1.95306 rpy=1.55156 -0.00000 1.57080, axis 0.00000 0.00000 1.00000, limit lower=-0.78500 upper=1.04700 effort=0.00000 velocity=0.00000
- added joint joint_l1_hip: type revolute, parent Internal-Frame-v121_link, child L1-v117_link, origin xyz=2.46389 2.58302 2.03634 rpy=-0.00000 -0.00000 -0.00000, axis 0.00000 0.00000 1.00000, limit lower=-0.78500 upper=0.78500 effort=0.00000 velocity=0.00000
- added joint joint_l2_hip: type revolute, parent Internal-Frame-v121_link, child L2-v117_link, origin xyz=-2.39531 2.58330 2.03634 rpy=0.00000 -0.00000 3.14159, axis 0.00000 0.00000 1.00000, limit lower=-0.78500 upper=0.78500 effort=0.00000 velocity=0.00000
- added joint joint_l3_foot: type revolute, parent L1-v117_link, child L3-v117_link, origin xyz=-0.93384 3.68844 -1.95242 rpy=1.57080 0.00000 1.57080, axis 0.00000 0.00000 1.00000, limit lower=-0.78500 upper=1.04700 effort=0.00000 velocity=0.00000
- added joint joint_l4_foot: type revolute, parent L2-v117_link, child L4-v117_link, origin xyz=0.63398 -4.70180 -1.66469 rpy=1.55975 0.00000 1.57080, axis 0.00000 0.00000 1.00000, limit lower=-0.78500 upper=1.04700 effort=0.00000 velocity=0.00000
- added joint joint_r1_hip: type revolute, parent Internal-Frame-v121_link, child R1-v117_link, origin xyz=2.46494 -2.51056 2.03634 rpy=-0.00000 0.00000 0.00000, axis 0.00000 0.00000 1.00000, limit lower=-0.78500 upper=0.78500 effort=0.00000 velocity=0.00000
- added joint joint_r2_hip: type revolute, parent Internal-Frame-v121_link, child R2-v117_link, origin xyz=-2.40342 -2.49865 2.03634 rpy=-0.00000 -0.00000 3.14159, axis 0.00000 0.00000 1.00000, limit lower=-0.78500 upper=0.78500 effort=0.00000 velocity=0.00000
- added joint joint_r4_foot: type revolute, parent R2-v117_link, child R4-v117_link, origin xyz=-0.95498 3.67349 -1.95620 rpy=1.55156 0.00000 1.57080, axis 0.00000 0.00000 1.00000, limit lower=-0.78500 upper=1.04700 effort=0.00000 velocity=0.00000

Commit message: feat: Add multi-robot dashboard support, visual SLAM, dual robot URDF, and unified robot firmware

File: urdf/unnamed/urdf/unnamed.urdf (robot description, URDF)
Before this commit: robot unnamed, 9 links, 8 joints
Links:
- link Internal-Frame-v121_link: mass None -> 0.28; geometry collision mesh filename=file:///home/sabo/Documents/learn_/Hardware/urdf/unnamed/me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 scale=1 1 1; visual mesh filename=file:///home/sabo/Documents/learn_/Hardware/urdf/unnamed/me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 scale=1 1 1
- link L1-v117_link: mass None -> 0.03; geometry collision mesh filename=file:///home/sabo/Documents/learn_/Hardware/urdf/unnamed/me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 scale=1 1 1; visual mesh filename=file:///home/sabo/Documents/learn_/Hardware/urdf/unnamed/me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 scale=1 1 1
- link L2-v117_link: mass None -> 0.03; geometry collision mesh filename=file:///home/sabo/Documents/learn_/Hardware/urdf/unnamed/me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 scale=1 1 1; visual mesh filename=file:///home/sabo/Documents/learn_/Hardware/urdf/unnamed/me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 scale=1 1 1
- link L3-v117_link: mass None -> 0.02; geometry collision mesh filename=file:///home/sabo/Documents/learn_/Hardware/urdf/unnamed/me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 scale=1 1 1; visual mesh filename=file:///home/sabo/Documents/learn_/Hardware/urdf/unnamed/me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 scale=1 1 1
- link L4-v117_link: mass None -> 0.02; geometry collision mesh filename=file:///home/sabo/Documents/learn_/Hardware/urdf/unnamed/me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 scale=1 1 1; visual mesh filename=file:///home/sabo/Documents/learn_/Hardware/urdf/unnamed/me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 scale=1 1 1
- link R1-v117_link: mass None -> 0.03; geometry collision mesh filename=file:///home/sabo/Documents/learn_/Hardware/urdf/unnamed/me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 scale=1 1 1; visual mesh filename=file:///home/sabo/Documents/learn_/Hardware/urdf/unnamed/me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 scale=1 1 1
- link R2-v117_link: mass None -> 0.03; geometry collision mesh filename=file:///home/sabo/Documents/learn_/Hardware/urdf/unnamed/me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 scale=1 1 1; visual mesh filename=file:///home/sabo/Documents/learn_/Hardware/urdf/unnamed/me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 scale=1 1 1
- link R3-v117_link: mass None -> 0.02; geometry collision mesh filename=file:///home/sabo/Documents/learn_/Hardware/urdf/unnamed/me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 scale=1 1 1; visual mesh filename=file:///home/sabo/Documents/learn_/Hardware/urdf/unnamed/me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 scale=1 1 1
- link R4-v117_link: mass None -> 0.02; geometry collision mesh filename=file:///home/sabo/Documents/learn_/Hardware/urdf/unnamed/me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 scale=1 1 1; visual mesh filename=file:///home/sabo/Documents/learn_/Hardware/urdf/unnamed/me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 scale=1 1 1
Joints:
- removed joint R3-v117_link_joint
- added joint joint_r3_foot: type revolute, parent R1-v117_link, child R3-v117_link, origin xyz=-0.009414 -0.036856 -0.019531 rpy=1.55156 0.00000 1.57080, axis 0 0 1, limit lower=-0.7854 upper=1.0472 effort=2.5 velocity=6.0
- joint joint_l1_hip: axis 0.00000 0.00000 1.00000 -> 0 0 1; limit lower=-0.78500 upper=0.78500 effort=0.00000 velocity=0.00000 -> lower=-0.7854 upper=0.7854 effort=2.5 velocity=6.0; origin xyz=2.46389 2.58302 2.03634 rpy=-0.00000 -0.00000 -0.00000 -> xyz=0.024639 0.025830 0.020363 rpy=0.00000 0.00000 0.00000
- joint joint_l2_hip: axis 0.00000 0.00000 1.00000 -> 0 0 1; limit lower=-0.78500 upper=0.78500 effort=0.00000 velocity=0.00000 -> lower=-0.7854 upper=0.7854 effort=2.5 velocity=6.0; origin xyz=-2.39531 2.58330 2.03634 rpy=0.00000 -0.00000 3.14159 -> xyz=-0.023953 0.025833 0.020363 rpy=0.00000 0.00000 3.14159
- joint joint_l3_foot: axis 0.00000 0.00000 1.00000 -> 0 0 1; limit lower=-0.78500 upper=1.04700 effort=0.00000 velocity=0.00000 -> lower=-0.7854 upper=1.0472 effort=2.5 velocity=6.0; origin xyz=-0.93384 3.68844 -1.95242 rpy=1.57080 0.00000 1.57080 -> xyz=-0.009338 0.036884 -0.019524 rpy=1.57080 0.00000 1.57080
- joint joint_l4_foot: axis 0.00000 0.00000 1.00000 -> 0 0 1; limit lower=-0.78500 upper=1.04700 effort=0.00000 velocity=0.00000 -> lower=-0.7854 upper=1.0472 effort=2.5 velocity=6.0; origin xyz=0.63398 -4.70180 -1.66469 rpy=1.55975 0.00000 1.57080 -> xyz=-0.009349 -0.036870 -0.019547 rpy=1.55975 0.00000 1.57080
- joint joint_r1_hip: axis 0.00000 0.00000 1.00000 -> 0 0 1; limit lower=-0.78500 upper=0.78500 effort=0.00000 velocity=0.00000 -> lower=-0.7854 upper=0.7854 effort=2.5 velocity=6.0; origin xyz=2.46494 -2.51056 2.03634 rpy=-0.00000 0.00000 0.00000 -> xyz=0.024649 -0.025106 0.020363 rpy=0.00000 0.00000 0.00000
- joint joint_r2_hip: axis 0.00000 0.00000 1.00000 -> 0 0 1; limit lower=-0.78500 upper=0.78500 effort=0.00000 velocity=0.00000 -> lower=-0.7854 upper=0.7854 effort=2.5 velocity=6.0; origin xyz=-2.40342 -2.49865 2.03634 rpy=-0.00000 -0.00000 3.14159 -> xyz=-0.024034 -0.024987 0.020363 rpy=0.00000 0.00000 3.14159
- joint joint_r4_foot: axis 0.00000 0.00000 1.00000 -> 0 0 1; limit lower=-0.78500 upper=1.04700 effort=0.00000 velocity=0.00000 -> lower=-0.7854 upper=1.0472 effort=2.5 velocity=6.0; origin xyz=-0.95498 3.67349 -1.95620 rpy=1.55156 0.00000 1.57080 -> xyz=-0.009550 0.036735 -0.019562 rpy=1.55156 0.00000 1.57080
