Commit message: feat: Add quadruped Dogu URDF, SMURF, Blender model, and Phobos fixes
- Add Dogu robot Blender model under dog/Dogu.blend
- Add generated quadruped URDF and SMURF kinematics under dog/unnamed/ and urdf/unnamed/
- Update servo calibration angles to 180 deg in servo_calibration.json
- Document Phobos add-on compatibility fixes in PROJECT_CONTEXT_README.md

File: urdf/unnamed/urdf/unnamed.urdf (robot description, URDF)
Before this commit: robot quard_bot, 9 links, 8 joints
Links:
- removed link Internal-Frame-v121_link
- removed link L1-v117_link
- removed link L2-v117_link
- removed link L3-v117_link
- removed link L4-v117_link
- removed link R1-v117_link
- removed link R2-v117_link
- removed link R3-v117_link
- removed link R4-v117_link
- added link Body_link; visual box size=2.23178 0.54200 0.35652
- added link Femurback-left_link
- added link Femurback-right_link
- added link Femurfront-left_link
- added link Femurfront-right_link
- added link Hipback-left_link
- added link Hipback-right_link
- added link Hipfront-left_link
- added link Hipfront-right_link
- added link TibiaLback-left_link
- added link TibiaLback-right_link
- added link TibiaLfront-left_link
- added link TibiaLfront-right_link
Joints:
- removed joint joint_l1_hip
- removed joint joint_l2_hip
- removed joint joint_l3_foot
- removed joint joint_l4_foot
- removed joint joint_r1_hip
- removed joint joint_r2_hip
- removed joint joint_r3_foot
- removed joint joint_r4_foot
- added joint Femurback-left-joint: type revolute, parent Hipback-left_link, child Femurback-left_link, origin xyz=0.20010 -0.63604 -0.09756 rpy=1.14190 1.57080 -0.44834, axis 0.00000 0.00000 1.00000, limit lower=-3.14000 upper=3.14000 effort=0.00000 velocity=0.00000
- added joint Femurback-right-joint: type revolute, parent Hipback-right_link, child Femurback-right_link, origin xyz=-0.19846 -0.64343 -0.04818 rpy=1.58477 1.57080 0.00000, axis 0.00000 0.00000 1.00000, limit lower=-3.14000 upper=3.14000 effort=0.00000 velocity=0.00000
- added joint Femurfront-left-joint: type revolute, parent Hipfront-left_link, child Femurfront-left_link, origin xyz=-0.20056 -0.63601 0.09831 rpy=1.34289 -1.57080 0.22791, axis 0.00000 0.00000 1.00000, limit lower=-3.14000 upper=3.14000 effort=0.00000 velocity=0.00000
- added joint Femurfront-right-joint: type revolute, parent Hipfront-right_link, child Femurfront-right_link, origin xyz=0.19846 -0.64343 0.04818 rpy=1.57080 -1.57080 0.00000, axis 0.00000 0.00000 1.00000, limit lower=-3.14000 upper=3.14000 effort=0.00000 velocity=0.00000
- added joint Hipback-left-joint: type revolute, parent Body_link, child Hipback-left_link, origin xyz=-1.01689 0.09211 -0.03398 rpy=-3.14159 1.57080 -0.00000, axis 0.00000 0.00000 1.00000, limit lower=-3.14000 upper=3.14000 effort=0.00000 velocity=0.00000
- added joint Hipback-right: type revolute, parent Body_link, child Hipback-right_link, origin xyz=-1.01689 -0.08910 -0.03466 rpy=0.00000 -1.57080 0.00000, axis 0.00000 0.00000 1.00000, limit lower=-3.14000 upper=3.14000 effort=0.00000 velocity=0.00000
- added joint Hipfront-left-joint: type revolute, parent Body_link, child Hipfront-left_link, origin xyz=0.87024 0.09211 -0.03398 rpy=-3.14159 -1.57080 0.00000, axis 0.00000 0.00000 1.00000, limit lower=-3.14000 upper=3.14000 effort=0.00000 velocity=0.00000
- added joint Hipfront-right-joint_: type revolute, parent Body_link, child Hipfront-right_link, origin xyz=0.87024 -0.08910 -0.03466 rpy=0.00000 1.57080 0.00000, axis 0.00000 0.00000 1.00000, limit lower=-3.14000 upper=3.14000 effort=0.00000 velocity=0.00000
- added joint TibiaLback-left-joint: type revolute, parent Femurback-left_link, child TibiaLback-left_link, origin xyz=0.56915 -0.03142 -0.07694 rpy=-0.03874 0.01647 0.01122, axis 0.00000 0.00000 1.00000, limit lower=-3.14000 upper=3.14000 effort=0.00000 velocity=0.00000
- added joint TibiaLback-right_joint: type revolute, parent Femurback-right_link, child TibiaLback-right_link, origin xyz=0.57104 0.00281 0.03004 rpy=-0.02291 0.02386 -0.00055, axis 0.00000 0.00000 1.00000, limit lower=-3.14000 upper=3.14000 effort=0.00000 velocity=0.00000
- added joint TibiaLfront-left-joint: type revolute, parent Femurfront-left_link, child TibiaLfront-left_link, origin xyz=0.56967 0.00379 0.01526 rpy=0.02448 0.00784 0.00019, axis 0.00000 0.00000 1.00000, limit lower=-3.14000 upper=3.14000 effort=0.00000 velocity=0.00000
- added joint TibiaLfront-right: type revolute, parent Femurfront-right_link, child TibiaLfront-right_link, origin xyz=0.56805 -0.00026 0.01632 rpy=-0.01047 0.00000 0.01252, axis 0.00000 0.00000 1.00000, limit lower=-3.14000 upper=3.14000 effort=0.00000 velocity=0.00000
